File: LED_chaser.kicad_sch (KiCad schematic)
At the start: 0 parts

Commit message: ve schematic
Parts:
- added C1: 10uF, LED_Chaser_Fp:CP_Radial_D5.0mm_P2.50mm, symbol LED_Chaser_Sch:C_Polarized
- added C2: 0.01uF, LED_Chaser_Fp:C_Disc_D5.0mm_W2.5mm_P2.50mm, symbol LED_Chaser_Sch:C
- added D1: LED_CLK, LED_Chaser_Fp:LED_D5.0mm, symbol LED_Chaser_Sch:LED
- added D10, D11, D2, D3, D4, D5, D6, D7, D8, D9: LED, LED_Chaser_Fp:LED_D5.0mm, symbol LED_Chaser_Sch:LED
- added J1: 9V_IN, LED_Chaser_Fp:PinHeader_1x02_P2.54mm_Vertical, symbol LED_Chaser_Sch:Conn_01x02
- added R1: 10k, LED_Chaser_Fp:R_Axial_DIN0207_L6.3mm_D2.5mm_P10.16mm_Horizontal, symbol LED_Chaser_Sch:R_US
- added R2, R3: 680R, LED_Chaser_Fp:R_Axial_DIN0207_L6.3mm_D2.5mm_P10.16mm_Horizontal, symbol LED_Chaser_Sch:R_US
- added RV1: 10k, LED_Chaser_Fp:Potentiometer_Bourns_3386P_Vertical, symbol LED_Chaser_Sch:R_Potentiometer
- added U1: NE555P, LED_Chaser_Fp:DIP-8_W7.62mm, symbol LED_Chaser_Sch:NE555P
- added U2: CD4017, LED_Chaser_Fp:DIP-16_W7.62mm, symbol LED_Chaser_Sch:4017
Connections:
- new net: R1.2, RV1.1, U1.7 (DISCH)
- new net: C1.1, RV1.2, RV1.3, U1.2 (TRIG), U1.6 (THRES)
- new net: D10.1 (K), D11.1 (K), D2.1 (K), D3.1 (K), D4.1 (K), D5.1 (K), D6.1 (K), D7.1 (K), D8.1 (K), D9.1 (K), R2.1
- new net: C2.1, U1.5 (CONT)
- new net: D1.1 (K), R3.1
- new net: D1.2 (A), U1.3 (OUT), U2.14 (CLK)
- new net +9V: J1.1 (Pin_1), R1.1, U1.4 (~{RST}), U1.8 (VCC), U2.16 (VDD)
- new net GND: C1.2, C2.2, J1.2 (Pin_2), R2.2, R3.2, U1.1 (GND), U2.13 (CKEN), U2.15 (Reset), U2.8 (VSS)
- new net Q0: D2.2 (A), U2.3 (Q0)
- new net Q1: D3.2 (A), U2.2 (Q1)
- new net Q2: D4.2 (A), U2.4 (Q2)
- new net Q3: D5.2 (A), U2.7 (Q3)
- new net Q4: D6.2 (A), U2.10 (Q4)
- new net Q5: D7.2 (A), U2.1 (Q5)
- new net Q6: D8.2 (A), U2.5 (Q6)
- new net Q7: D9.2 (A), U2.6 (Q7)
- new net Q8: D10.2 (A), U2.9 (Q8)
- new net Q9: D11.2 (A), U2.11 (Q9)
- no-connect marks 0 -> 1
Other:
- company: (none) -> HUST - ET2021
- title: (none) -> Mach LED Chay Duoi 555 - CD4017

Commit message: Tao thu vien linh kien va ve xong schematic mach LED chaser
Other:
- moved on the sheet: C2
